Commit message: update

File: description/robot.xacro (robot description, xacro)
@@ -1,5 +1,5 @@
 <?xml version="1.0"?>
 <robot xmlns:xacro="http://www.ros.org/wiki/xacro" name="robot">
-    <xacro:property name="path"                 value="robot_system" />
+    <xacro:property name="path"                 value="robot_control" />
     <xacro:property name="chassis_length"       value="1.004" />
     <xacro:property name="chassis_length_mid"   value="0.6" />
